File: EDA/ISA-Card/ISA-Card.kicad_pcb (KiCad board)
At the start: 2 copper layers, 139.7 x 101.6 mm, 57 parts, among them J1 Floppy 1, J2 Floppy 2, J3 Floppy 3, J4 Floppy 4, J5 SERIAL, U1 82077AA, U10 74AHCT138, U2 82077AA, U3 16C550, U4 GD75232N, U5 Flash ROM, U6 EEPROM, U7 74HCT688, U8 74AHCT138, U9 74AHCT138, X1 24MHz, X2 1.8432MHz

Commit message: Schematic done except response signal, PCB started
Parts:
- removed C10, C11, C12, C13, C14, C15, C16, C17: 100nF, My_Components:Cap_Cer_508
- removed C18, C19, C20, C22, C23: 10uF, My_Components:Cap_Elec_Radial_6.3mm
- removed HOLE1: HOLE, MountingHole:MountingHole_3.2mm_M3_Pad_Via
- removed J1: Floppy 1, My_Components:Conn_Pin_Header_17x2_2.54mm_Shrouded
- removed J2: Floppy 2, My_Components:Conn_Pin_Header_17x2_2.54mm_Shrouded
- removed J3: Floppy 3, My_Components:Conn_Pin_Header_17x2_2.54mm_Shrouded
- removed J4: Floppy 4, My_Components:Conn_Pin_Header_17x2_2.54mm_Shrouded
- removed J5: SERIAL, My_Components:Conn_Dsub_DE9M
- removed JP1: IO_CONFIG, My_Components:Conn_Pin_Header_6x2_2.54mm
- removed JP2: FDC2_IRQ, My_Components:Conn_Pin_Header_6x2_2.54mm
- removed JP3: FDC2_DMA, My_Components:Conn_Pin_Header_6x2_2.54mm
- removed JP4: UART_IRQ, My_Components:Conn_Pin_Header_5x1_2.54mm
- removed JP5: ROM_CONFIG, My_Components:Conn_Pin_Header_7x2_2.54mm
- removed JP6: Floppy 1 - 5V, My_Components:Conn_Pin_Header_2x1_2.54mm_NoKey
- removed JP7: Floppy 2 - 5V, My_Components:Conn_Pin_Header_2x1_2.54mm_NoKey
- removed JP8: Floppy 3 - 5V, My_Components:Conn_Pin_Header_2x1_2.54mm_NoKey
- removed JP9: Floppy 4 - 5V, My_Components:Conn_Pin_Header_2x1_2.54mm_NoKey
- removed REF**: KiCad-Logo2_5mm_SilkScreen, Symbol:KiCad-Logo2_5mm_SilkScreen
- removed REF**: OSHW-Logo2_7.3x6mm_SilkScreen, Symbol:OSHW-Logo2_7.3x6mm_SilkScreen
- removed RN1, RN2: 1k, My_Components:Conn_SIL6
- removed RN3, RN4: 10k, My_Components:Conn_SIL6
- removed U1, U2: 82077AA, My_Components:IC_PLCC68_TH
- removed U10, U8, U9: 74AHCT138, My_Components:IC_DIP16_300
- removed U3: 16C550, My_Components:IC_PLCC44_TH
- removed U4: GD75232N, My_Components:IC_DIP20_300
- removed U5: Flash ROM, My_Components:IC_DIP32_600
- removed U6: EEPROM, My_Components:IC_DIP28_600
- removed U7: 74HCT688, My_Components:IC_DIP20_300
- removed X1: 24MHz, My_Components:OSC_Half_Can_DIP8
- added R1: R, Resistor_SMD:R_0603_1608Metric, F.Cu at (59.5, 12.4)
- added R10: R, Resistor_SMD:R_0603_1608Metric, F.Cu at (55.5, 12.4)
- added R11: R, Resistor_SMD:R_0603_1608Metric, F.Cu at (143.7, -55.9)
- added R12: R, Resistor_SMD:R_0603_1608Metric, F.Cu at (77.2, 9.86)
- added R13: R, Resistor_SMD:R_0603_1608Metric, F.Cu at (131.7, -45.8)
- added R14: R, Resistor_SMD:R_0603_1608Metric, F.Cu at (131.7, -55.9)
- added R15: R, Resistor_SMD:R_0603_1608Metric, F.Cu at (67.6, 12.4)
- added R16: R, Resistor_SMD:R_0603_1608Metric, F.Cu at (71.6, 12.4)
- added R2: R, Resistor_SMD:R_0603_1608Metric, F.Cu at (135.7, -53.3)
- added R3: R, Resistor_SMD:R_0603_1608Metric, F.Cu at (55.5, -12.0)
- added R4: R, Resistor_SMD:R_0603_1608Metric, F.Cu at (81.2, 7.35)
- added R5: R, Resistor_SMD:R_0603_1608Metric, F.Cu at (120.8, -36.5)
- added R6: R, Resistor_SMD:R_0603_1608Metric, F.Cu at (131.7, -50.8)
- added R7: R, Resistor_SMD:R_0603_1608Metric, F.Cu at (135.7, -55.9)
- added R8: R, Resistor_SMD:R_0603_1608Metric, F.Cu at (88.1, 4.85)
- added R9: R, Resistor_SMD:R_0603_1608Metric, F.Cu at (135.7, -50.8)
- added U7101: 74HCT245, Package_DIP:DIP-20_W7.62mm, F.Cu at (247.0, -5.71)
- added U7102: 74HCT244, Package_DIP:DIP-20_W7.62mm, F.Cu at (219.1, -5.71)
- added U7104: 74HCT138, Package_DIP:DIP-16_W7.62mm, F.Cu at (194.3, -5.71)
- added U7105: 74HCT138, Package_DIP:DIP-16_W7.62mm, F.Cu at (168.3, -6.35)
- added U7106: 74LS08, Package_DIP:DIP-14_W7.62mm, F.Cu at (213.4, -21.6)
- added U7107: 74LS32, Package_DIP:DIP-14_W7.62mm, F.Cu at (168.3, -21.6)
- added U7108: 74LS32, Package_DIP:DIP-14_W7.62mm, F.Cu at (168.3, -36.2)
- added U7109: 74HC368, Package_DIP:DIP-16_W7.62mm, F.Cu at (214.0, -51.4)
- added U7110: 74HC04, Package_DIP:DIP-14_W7.62mm, F.Cu at (190.5, -51.4)
- added U7111: 74HC125, Package_DIP:DIP-14_W7.62mm, F.Cu at (214.0, -36.2)
- added U7112: 74HC74, Package_DIP:DIP-14_W7.62mm, F.Cu at (168.3, -51.4)
- added U7113: 74HC74, Package_DIP:DIP-14_W7.62mm, F.Cu at (191.1, -36.2)
- added U7114: 74HC4024, Package_DIP:DIP-14_W7.62mm, F.Cu at (211.5, -70.5)
- added U7115: 74HC4024, Package_DIP:DIP-14_W7.62mm, F.Cu at (168.3, -70.5)
- added U7116: 74HC595, Package_DIP:DIP-16_W7.62mm, F.Cu at (239.4, -51.4)
- added U7117: 74HC595, Package_DIP:DIP-16_W7.62mm, F.Cu at (240.1, -36.2)
- added U7118: 74HC595, Package_DIP:DIP-16_W7.62mm, F.Cu at (239.4, -21.6)
- added U7119: 8251, Package_DIP:DIP-28_W15.24mm_Socket, F.Cu at (248.9, -66.7)
- added U7120: 26LS31, Package_DIP:DIP-16_W7.62mm, F.Cu at (263.5, -51.4)
- added U7121: 26LS32, Package_DIP:DIP-16_W7.62mm, F.Cu at (264.2, -36.2)
- added X-TAL1: Crystal, Crystal:Crystal_HC52-U_Horizontal, F.Cu at (197.5, -67.2)
- added X3: DB15_Female, Connector_Dsub:DSUB-15_Female_Horizontal_P2.77x2.84mm_EdgePinOffset7.70mm_Housed_MountingHolesOffset9.12mm, F.Cu at (288.9, -29.8)
- added X5: Conn_02x08_Counter_Clockwise, Connector_PinHeader_2.54mm:PinHeader_2x08_P2.54mm_Vertical, F.Cu at (288.9, -87.0)
- C1, C2: value 4.7nF -> C; footprint My_Components:Cap_Cer_508 -> Capacitor_SMD:C_0603_1608Metric
- C3, C4, C5, C6, C7, C8: value 100nF -> C; footprint My_Components:Cap_Cer_508 -> Capacitor_SMD:C_0603_1608Metric
- C9: value 100nF -> C; footprint My_Components:Cap_Cer_508 -> Capacitor_THT:CP_Radial_D10.0mm_P5.00mm
- X2: value 1.8432MHz -> Conn_02x04_Counter_Clockwise; footprint My_Components:OSC_Half_Can_DIP8 -> Connector_PinHeader_2.54mm:PinHeader_2x04_P2.54mm_Vertical
- moved C9 219.7 mm to (238.8, -79.2)
- moved C8 186.1 mm to (131.7, -48.3)
- moved C3 138.3 mm to (55.5, -9.46), turned to 0 degrees
- moved C1 138.2 mm to (139.7, -53.3), turned to 0 degrees
- moved C2 136.7 mm to (131.7, -53.3), turned to 0 degrees
- moved C4 132.8 mm to (139.7, -55.9), turned to 0 degrees
- moved C7 124.9 mm to (63.5, 12.4), turned to 0 degrees
- moved C5 89.5 mm to (77.2, 7.35), turned to 0 degrees
- moved X2 84.6 mm to (196.9, -23.5), turned to 90 degrees
- moved HOLE2 74.3 mm to (207.0, 63.5)
- moved C6 67.8 mm to (75.6, 12.4), turned to 0 degrees
Connections:
- BUS1 pad 10: GND -> unconnected-(BUS1-Pad10)
- BUS1 pad 11: /~MEMW -> unconnected-(BUS1-Pad11)
- BUS1 pad 12: /~MEMR -> unconnected-(BUS1-Pad12)
- BUS1 pad 13: /~IOW -> /~{IOW}
- BUS1 pad 14: /~IOR -> /~{IOR}
- BUS1 pad 15: /~DACK3 -> /~{DACK3}
- BUS1 pad 17: /~DACK1 -> unconnected-(BUS1-Pad17)
- BUS1 pad 18: /DRQ1 -> unconnected-(BUS1-Pad18)
- BUS1 pad 21: /IRQ7 -> unconnected-(BUS1-Pad21)
- BUS1 pad 22: /IRQ6 -> unconnected-(BUS1-Pad22)
- BUS1 pad 23: /IRQ5 -> unconnected-(BUS1-Pad23)
- BUS1 pad 24: /IRQ4 -> unconnected-(BUS1-Pad24)
- BUS1 pad 25: /IRQ3 -> unconnected-(BUS1-Pad25)
- BUS1 pad 26: /~DACK2 -> unconnected-(BUS1-Pad26)
- BUS1 pad 27: /TC -> unconnected-(BUS1-Pad27)
- BUS1 pad 29: VCC -> unconnected-(BUS1-Pad29)
- BUS1 pad 31: GND -> unconnected-(BUS1-Pad31)
- BUS1 pad 4: /IRQ2 -> unconnected-(BUS1-Pad4)
- BUS1 pad 43: /A19 -> unconnected-(BUS1-Pad43)
- BUS1 pad 44: /A18 -> unconnected-(BUS1-Pad44)
- BUS1 pad 45: /A17 -> unconnected-(BUS1-Pad45)
- BUS1 pad 46: /A16 -> unconnected-(BUS1-Pad46)
- BUS1 pad 47: /A15 -> unconnected-(BUS1-Pad47)
- BUS1 pad 48: /A14 -> unconnected-(BUS1-Pad48)
- BUS1 pad 49: /A13 -> unconnected-(BUS1-Pad49)
- BUS1 pad 50: /A12 -> unconnected-(BUS1-Pad50)
- BUS1 pad 51: /A11 -> unconnected-(BUS1-Pad51)
- BUS1 pad 52: /A10 -> unconnected-(BUS1-Pad52)
- BUS1 pad 6: /DRQ2 -> unconnected-(BUS1-Pad6)
- BUS1 pad 7: -12V -> unconnected-(BUS1-Pad7)
- BUS1 pad 9: +12V -> unconnected-(BUS1-Pad9)
- C1 pad 1: Net-(C1-Pad1) -> unconnected-(C1-Pad1)
- C1 pad 2: Net-(C1-Pad2) -> GND
- C2 pad 1: Net-(C2-Pad1) -> VCC
- C2 pad 2: Net-(C2-Pad2) -> GND
- C4 pad 1: VCC -> GND
- C4 pad 2: GND -> Net-(U7108-Pad2)
- C5 pad 1: VCC -> GND
- C5 pad 2: GND -> Net-(U7110-Pad11)
- C6 pad 1: VCC -> GND
- C6 pad 2: GND -> Net-(U7110-Pad10)
- C7 pad 1: VCC -> Net-(U7114-Pad1)
- C8 pad 1: VCC -> GND
- C8 pad 2: GND -> VCC
- C9 pad 1: VCC -> GND
- C9 pad 2: GND -> VCC
- X2 pad 4: GND -> Net-(U7104-Pad11)
- X2 pad 5: /UART_CLK -> Net-(U7105-Pad5)
- X2 pad 8: VCC -> Net-(U7105-Pad5)
Routing:
- net GND: track 1668.5 -> 0.00 mm, vias 42 -> 0
- net VCC: track 873.1 -> 0.00 mm, vias 8 -> 0
- net /A0: track 240.8 -> 0.00 mm, vias 3 -> 0
- net /A1: track 235.1 -> 0.00 mm, vias 3 -> 0
- net /A2: track 214.9 -> 0.00 mm, vias 3 -> 0
- net /~UART_CS: track 195.6 -> 0.00 mm, vias 2 -> 0
- net /RESETDRV: track 181.7 -> 0.00 mm, vias 1 -> 0
- net /D1: track 176.6 -> 0.00 mm, vias 2 -> 0
- net /~IOW: track 175.5 -> 0.00 mm, vias 2 -> 0
- net /~IOR: track 174.3 -> 0.00 mm, vias 2 -> 0
- net /D0: track 173.9 -> 0.00 mm, vias 2 -> 0
- net /D5: track 163.9 -> 0.00 mm, vias 2 -> 0
- net /D3: track 163.4 -> 0.00 mm, vias 2 -> 0
- net /D2: track 159.7 -> 0.00 mm, vias 2 -> 0
- net /D4: track 159.5 -> 0.00 mm, vias 5 -> 0
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- removed copper zone on B.Cu, net GND
- removed copper zone on F.Cu, net GND
Other:
- board size 139.7 x 101.6 mm -> 146.1 x 101.6 mm
- net class Default removed
- net class FLOPPY_VCC removed
- net class GND removed
- net class VCC removed
- board text removed: "!"
- board text removed: "32KB"
- board text removed: "A15"
- board text removed: "A16"
- board text removed: "A17"
- board text removed: "Address 0xC0000 0xC8000 0xD0000 0xD8000 0xE0000 0xE8000"
- board text removed: "COM1"
- board text removed: "COM2"
- board text removed: "COM3"
- board text removed: "COM4"
- board text removed: "Copyright (C) 2021 Sergey Kiselev"
- board text removed: "DMA1"
- board text removed: "DMA2"
- board text removed: "DMA3"
- board text removed: "Designed in Oregon"
- board text removed: "Enable"
- board text removed: "FDC1"
- board text removed: "FDC2"
- board text removed: "IRQ2"
- board text removed: "IRQ3"
- board text removed: "IRQ4"
- board text removed: "IRQ5"
- board text removed: "IRQ6"
- board text removed: "IRQ7"
- board text removed: "JP1 - I/O Ports Configuration JP1.1 - Enable Primary FDC at 0x3F0 JP1.2 - Enable Secondary FDC at 0x370 JP1.3 - Enable UART at 0x3F8 (COM1)"
- board text removed: "JP1.4 - Enable UART at 0x2F8 (COM2) JP1.5 - Enable UART at 0x3E8 (COM3) JP1.6 - Enable UART at 0x2E8 (COM4) Set only one of JP1.3 - JP1.6 jumpers"
- board text removed: "JP2 - Sec. FDC IRQ Configuration JP2.1 - ON: IRQ6 JP2.2 - ON: IRQ4 JP2.3 - ON: IRQ3 JP2.4 - ON: IRQ5 JP2.5 - ON: IRQ7 JP2.6 - ON: IRQ2 Set only one of JP2.x jumpers"
- board text removed: "JP3 - Sec. FDC DMA Configuration JP3.1 and JP3.2 - ON: DMA Channel 2* JP3.3 and JP3.4 - ON: DMA Channel 1 JP3.5 and JP3.6 - ON: DMA Channel 3 Set only one pair of JP3.1-JP3.6 jumpers"
- board text removed: "JP4 - UART IRQ Configuration JP4.1 - ON: IRQ4 (COM1, COM3) JP4.2 - ON: IRQ3 (COM2, COM4) JP4.3 - ON: IRQ5"
- board text removed: "JP4.4 - ON: IRQ7 JP4.5 - ON: IRQ2 Set only one of JP4.x jumpers"
- board text removed: "JP5 - BIOS Extension ROM Configuration JP5.1 - OFF/ON: Disable/Enable ROM JP5.5 and JP5.6 - OFF: 8 KiB ROM (28C64); JP5.5 and JP5.6 - ON: 32 KiB ROM (28C256, 39SF010) JP5.7 - OFF/ON: Disable/Enable EEPROM write"
- board text removed: "JP5.2 - JP.4 - BIOS Extension ROM Address"
- board text removed: "JP5.2 OFF OFF OFF OFF ON ON"
- board text removed: "JP5.3 OFF OFF ON ON OFF OFF"
- board text removed: "JP5.4 OFF ON OFF ON OFF ON"
- board text removed: "Licensed under CERN-OHL-S Design files and documentation: github.com/skiselev/monster-fdc"
- board text removed: "Monster FDC Version 1.0"
- board text removed: "WARNING: Install JP6-JP9 jumpers only with PS/2 floppy drives that are powered by pin 3"
- board text removed: "Write"
- board text removed: "www.malinov.com"

Commit message: PCB Major Progress
Parts:
- added HOLE2: HOLE, MountingHole:MountingHole_3.2mm_M3_Pad_Via, F.Cu at (200.0, 85.1)
- added HOLE2: HOLE, MountingHole:MountingHole_3.2mm_M3_Pad_Via, F.Cu at (78.1, 57.1)
- C1, C2, C3, C4, C5, C6, C7, C8: footprint Capacitor_SMD:C_0603_1608Metric -> Capacitor_SMD:C_1206_3216Metric
- C9: value C -> C_Polarized
- R1, R10, R11, R12, R13, R14, R15, R16, R2, R3, R4, R5, R6, R7, R8, R9: footprint Resistor_SMD:R_0603_1608Metric -> Resistor_SMD:R_1206_3216Metric
- moved R10 204.1 mm to (223.5, 128.4), turned to 90 degrees
- moved R1 198.6 mm to (223.5, 124.4), turned to 90 degrees
- moved C7 193.0 mm to (223.5, 120.4), turned to 90 degrees
- moved R15 187.4 mm to (223.5, 116.4), turned to 90 degrees
- moved C3 187.3 mm to (215.3, 88.3)
- moved R3 187.3 mm to (215.3, 85.8)
- moved R16 181.9 mm to (223.5, 112.4), turned to 90 degrees
- moved C6 176.3 mm to (223.5, 108.4), turned to 90 degrees
- moved R12 173.3 mm to (220.9, 106.7), turned to 90 degrees
- moved C5 172.7 mm to (218.4, 106.7), turned to 90 degrees
- moved X5 172.0 mm to (198.1, 59.1)
- moved R11 169.5 mm to (232.9, 88.3), turned to 180 degrees
- moved U7105 168.2 mm to (77.5, 135.2)
- moved U7107 168.2 mm to (77.5, 120.0)
- moved U7118 168.2 mm to (148.6, 120.0)
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Connections:
- net Net-(U7107-Pad1) renamed /Data Clock HV
- net Net-(U7121-Pad11) renamed /Response
- C9 pad 1: GND -> VCC
- C9 pad 2: VCC -> GND
- U7105 pad 5: Net-(U7105-Pad5) -> /Port Selection
- U7107 pad 5: Net-(U7105-Pad5) -> /Port Selection
- U7109 pad 12: Net-(U7109-Pad12) -> /Attention
- U7109 pad 5: Net-(U7109-Pad5) -> /Data
- U7109 pad 9: Net-(U7109-Pad12) -> /Attention
- U7111 pad 9: Net-(U7111-Pad9) -> /Command
- U7113 pad 12: VCC -> GND
- U7116 pad 14: Net-(U7109-Pad5) -> /Data
- U7118 pad 14: Net-(U7109-Pad12) -> /Attention
- U7119 pad 19: Net-(U7111-Pad9) -> /Command
- U7119 pad 22: Net-(U7109-Pad12) -> /Attention
- U7119 pad 25: Net-(U7119-Pad25) -> /Data Clock LV
- U7119 pad 9: Net-(U7119-Pad25) -> /Data Clock LV
- U7120 pad 9: Net-(U7111-Pad9) -> /Command
- U7121 pad 12: Net-(U7119-Pad25) -> /Data Clock LV
- U7121 pad 13: Net-(U7109-Pad12) -> /Attention
- U7121 pad 5: Net-(U7109-Pad5) -> /Data
- X2 pad 2: Net-(U7104-Pad14) -> /Port Selection
- X2 pad 3: Net-(U7104-Pad12) -> Net-(U7104-Pad14)
- X2 pad 4: Net-(U7104-Pad11) -> /Port Selection
- X2 pad 5: Net-(U7105-Pad5) -> Net-(U7104-Pad12)
- X2 pad 6: Net-(U7105-Pad5) -> /Port Selection
- X2 pad 7: Net-(U7105-Pad5) -> Net-(U7104-Pad11)
- X2 pad 8: Net-(U7105-Pad5) -> /Port Selection
- X5 pad 2: Net-(U7111-Pad9) -> GND
- X5 pad 3: Net-(U7109-Pad5) -> /Command
- X5 pad 4: Net-(U7119-Pad25) -> GND
- X5 pad 5: Net-(U7109-Pad12) -> /Data
- X5 pad 7: unconnected-(X5-Pad7) -> /Data Clock LV
- X5 pad 8: GND -> unconnected-(X5-Pad8)
- X5 pad 9: GND -> /Attention
Routing:
- net GND: track 0.00 -> 756.0 mm, vias 0 -> 11
- net VCC: track 0.00 -> 664.9 mm, vias 0 -> 9
- net Net-(U7110-Pad12): track 0.00 -> 197.3 mm, vias 0 -> 8
- net /Data Clock HV: track 0.00 -> 166.7 mm, vias 0 -> 5
- net Net-(U7108-Pad1): track 0.00 -> 145.0 mm, vias 0 -> 5
- net /MDB1: track 0.00 -> 144.7 mm, vias 0 -> 5
- net Net-(U7105-Pad15): track 0.00 -> 140.4 mm, vias 0 -> 3
- net Net-(U7101-Pad1): track 0.00 -> 134.7 mm, vias 0 -> 3
- net Net-(U7108-Pad11): track 0.00 -> 133.9 mm, vias 0 -> 8
- net /MDB2: track 0.00 -> 126.3 mm, vias 0 -> 4
- net /Data: track 0.00 -> 114.0 mm, vias 0 -> 4
- net /RESETDRV: track 0.00 -> 110.8 mm, vias 0 -> 4
- net Net-(U7102-Pad18): track 0.00 -> 108.5 mm, vias 0 -> 1
- net /MDB3: track 0.00 -> 106.3 mm, vias 0 -> 3
- net /MDB4: track 0.00 -> 102.6 mm, vias 0 -> 4
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Other:
- board size 146.1 x 101.6 mm -> 138.4 x 98.4 mm

Commit message: PCB Primary Routing finished, except 2 traces
Parts:
- C1, C2, C3, C4, C5, C6, C7, C8, R1, R10, R11, R12, R13, R14, R15, R16, R2, R3, R4, R5, R6, R7, R8, R9: moved to B.Cu
- moved R14 135.1 mm to (187.5, 125.7), turned to 180 degrees
- moved R13 132.1 mm to (187.4, 122.4), turned to 180 degrees
- moved C6 130.4 mm to (100.6, 65.0)
- moved R4 130.2 mm to (88.3, 102.2), turned to 0 degrees
- moved R9 127.4 mm to (187.3, 113.0), turned to 180 degrees
- moved R1 120.4 mm to (105.4, 101.0)
- moved R5 118.2 mm to (180.3, 116.2), turned to 180 degrees
- moved R6 117.5 mm to (172.1, 119.4), turned to 180 degrees
- moved C5 115.9 mm to (110.2, 65.0)
- moved R7 115.6 mm to (172.1, 122.6), turned to 180 degrees
- moved C7 115.3 mm to (118.7, 72.4), turned to -90 degrees
- moved R3 100.6 mm to (115.6, 72.4), turned to -90 degrees
- moved C8 87.6 mm to (139.1, 66.7), turned to 90 degrees
- moved C2 87.1 mm to (141.0, 116.2), turned to -90 degrees
- moved C3 75.4 mm to (141.0, 101.0), turned to -90 degrees
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Connections:
- C1 pad 1: unconnected-(C1-Pad1) -> VCC
- X-TAL1 pad 1: Net-(C6-Pad2) -> Net-(C5-Pad2)
- X-TAL1 pad 2: Net-(C5-Pad2) -> Net-(C6-Pad2)
Routing:
- net /Attention: track 27.6 -> 179.8 mm, vias 1 -> 7
- net Net-(U7115-Pad9): track 0.00 -> 147.3 mm, vias 0 -> 4
- net Net-(U7105-Pad14): track 77.9 -> 183.3 mm, vias 1 -> 5
- net /Data Clock LV: track 0.00 -> 88.0 mm, vias 0 -> 3
- net /Command: track 25.7 -> 111.6 mm, vias 0 -> 3
- net Net-(U7107-Pad12): track 69.6 -> 146.4 mm
- net Net-(U7108-Pad8): track 47.8 -> 122.6 mm, vias 0 -> 2
- net GND: track 756.0 -> 827.3 mm, vias 11 -> 26
- net Net-(U7101-Pad1): track 134.7 -> 200.8 mm, vias 3 -> 5
- net /Attention-: track 0.00 -> 65.1 mm, vias 0 -> 3
- net /Response: track 0.00 -> 61.9 mm, vias 0 -> 4
- net Net-(U7114-Pad12): track 0.00 -> 59.7 mm, vias 0 -> 1
- net VCC: track 664.9 -> 724.2 mm, vias 9 -> 18
- net /Data-: track 0.00 -> 57.5 mm, vias 0 -> 1
- net /Command-: track 0.00 -> 57.1 mm, vias 0 -> 1
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
Commit message: update readme
Parts:
- U7119: footprint Package_DIP:DIP-28_W15.24mm_Socket -> Package_DIP:DIP-28_W15.24mm
Changed lines of the file:
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@@
     )
   )
-  (footprint "Package_DIP:DIP-28_W15.24mm_Socket" (layer "F.Cu")
+  (footprint "Package_DIP:DIP-28_W15.24mm" (layer "F.Cu")
     (at 158.1 74.3 90)
-    (descr "28-lead though-hole mounted DIP package, row spacing 15.24 mm (600 mils), Socket")
-    (tags "THT DIP DIL PDIP 2.54mm 15.24mm 600mil Socket")
+    (descr "28-lead though-hole mounted DIP package, row spacing 15.24 mm (600 mils)")
+    (tags "THT DIP DIL PDIP 2.54mm 15.24mm 600mil")
     (property "Sheetfile" "ISA-Card.kicad_sch")
     (property "Sheetname" "")
@@
       (effects (font (size 1 1) (thickness 0.15)))
     )
+    (fp_line (start 1.16 -1.33) (end 1.16 34.35) (layer "F.SilkS") (width 0.12))
+    (fp_line (start 14.08 -1.33) (end 8.62 -1.33) (layer "F.SilkS") (width 0.12))
+    (fp_line (start 1.16 34.35) (end 14.08 34.35) (layer "F.SilkS") (width 0.12))
     (fp_line (start 14.08 34.35) (end 14.08 -1.33) (layer "F.SilkS") (width 0.12))
-    (fp_line (start -1.33 -1.39) (end -1.33 34.41) (layer "F.SilkS") (width 0.12))
-    (fp_line (start 16.57 34.41) (end 16.57 -1.39) (layer "F.SilkS") (width 0.12))
-    (fp_line (start 14.08 -1.33) (end 8.62 -1.33) (layer "F.SilkS") (width 0.12))
-    (fp_line (start 1.16 -1.33) (end 1.16 34.35) (layer "F.SilkS") (width 0.12))
     (fp_line (start 6.62 -1.33) (end 1.16 -1.33) (layer "F.SilkS") (width 0.12))
-    (fp_line (start 16.57 -1.39) (end -1.33 -1.39) (layer "F.SilkS") (width 0.12))
-    (fp_line (start 1.16 34.35) (end 14.08 34.35) (layer "F.SilkS") (width 0.12))
-    (fp_line (start -1.33 34.41) (end 16.57 34.41) (layer "F.SilkS") (width 0.12))
     (fp_arc (start 8.62 -1.33) (mid 7.62 -0.33) (end 6.62 -1.33) (layer "F.SilkS") (width 0.12))
-    (fp_line (start -1.55 34.65) (end 16.8 34.65) (layer "F.CrtYd") (width 0.05))
-    (fp_line (start 16.8 34.65) (end 16.8 -1.6) (layer "F.CrtYd") (width 0.05))
-    (fp_line (start -1.55 -1.6) (end -1.55 34.65) (layer "F.CrtYd") (width 0.05))
-    (fp_line (start 16.8 -1.6) (end -1.55 -1.6) (layer "F.CrtYd") (width 0.05))
-    (fp_line (start 14.985 -1.27) (end 14.985 34.29) (layer "F.Fab") (width 0.1))
-    (fp_line (start 16.51 34.35) (end 16.51 -1.33) (layer "F.Fab") (width 0.1))
-    (fp_line (start 0.255 34.29) (end 0.255 -0.27) (layer "F.Fab") (width 0.1))
-    (fp_line (start -1.27 -1.33) (end -1.27 34.35) (layer "F.Fab") (width 0.1))
-    (fp_line (start 0.255 -0.27) (end 1.255 -1.27) (layer "F.Fab") (width 0.1))
+    (fp_line (start -1.05 34.55) (end 16.3 34.55) (layer "F.CrtYd") (width 0.05))
+    (fp_line (start 16.3 34.55) (end 16.3 -1.55) (layer "F.CrtYd") (width 0.05))
+    (fp_line (start -1.05 -1.55) (end -1.05 34.55) (layer "F.CrtYd") (width 0.05))
+    (fp_line (start 16.3 -1.55) (end -1.05 -1.55) (layer "F.CrtYd") (width 0.05))
     (fp_line (start 14.985 34.29) (end 0.255 34.29) (layer "F.Fab") (width 0.1))
     (fp_line (start 1.255 -1.27) (end 14.985 -1.27) (layer "F.Fab") (width 0.1))
-    (fp_line (start -1.27 34.35) (end 16.51 34.35) (layer "F.Fab") (width 0.1))
-    (fp_line (start 16.51 -1.33) (end -1.27 -1.33) (layer "F.Fab") (width 0.1))
+    (fp_line (start 14.985 -1.27) (end 14.985 34.29) (layer "F.Fab") (width 0.1))
+    (fp_line (start 0.255 -0.27) (end 1.255 -1.27) (layer "F.Fab") (width 0.1))
+    (fp_line (start 0.255 34.29) (end 0.255 -0.27) (layer "F.Fab") (width 0.1))
     (pad "1" thru_hole rect (at 0 0 90) (size 1.6 1.6) (drill 0.8) (layers *.Cu *.Mask)
       (net 77 "/MDB6") (pinfunction "D2") (pintype "bidirectional"))
@@
     (pad "28" thru_hole oval (at 15.24 0 90) (size 1.6 1.6) (drill 0.8) (layers *.Cu *.Mask)
       (net 78 "/MDB7") (pinfunction "D1") (pintype "bidirectional"))
-    (model "${KICAD6_3DMODEL_DIR}/Package_DIP.3dshapes/DIP-28_W15.24mm_Socket.wrl"
+    (model "${KICAD6_3DMODEL_DIR}/Package_DIP.3dshapes/DIP-28_W15.24mm.wrl"
       (offset (xyz 0 0 0))
       (scale (xyz 1 1 1))
@@
   (segment (start 193.675 68.491834) (end 185.966834 68.491834) (width 1) (layer "F.Cu") (net 24))
   (segment (start 76.157265 103.601396) (end 75.692 104.066661) (width 0.4) (layer "F.Cu") (net 24))
+  (segment (start 75.692 106.172) (end 76.2 106.68) (width 0.4) (layer "F.Cu") (net 24))
   (segment (start 185.674 133.35) (end 179.07 133.35) (width 1) (layer "F.Cu") (net 24))
   (segment (start 94.605 120.005) (end 92.07 120.005) (width 0.4) (layer "F.Cu") (net 24))
@@
   (segment (start 179.07 135.255) (end 179.07 133.35) (width 0.4) (layer "F.Cu") (net 24))
   (segment (start 92.07 104.765) (end 92.07 102.875) (width 0.4) (layer "F.Cu") (net 24))
-  (segment (start 90.932 106.68) (end 90.932 106.538) (width 0.4) (layer "F.Cu") (net 24))
   (segment (start 120.65 133.35) (end 94.615 133.35) (width 1) (layer "F.Cu") (net 24))
   (segment (start 123.913166 68.491834) (end 110.324166 68.491834) (width 1) (layer "F.Cu") (net 24))
@@
   (segment (start 166.385 89.535) (end 166.385 87.645) (width 0.4) (layer "F.Cu") (net 24))
   (segment (start 119.126 87.63) (end 114.935 87.63) (width 1) (layer "F.Cu") (net 24))
-  (segment (start 75.692 106.172) (end 76.2 106.68) (width 0.4) (layer "F.Cu") (net 24))
   (segment (start 136.52 70.475) (end 136.52 68.575) (width 0.4) (layer "F.Cu") (net 24))
   (segment (start 114.93 104.775) (end 114.93 102.875) (width 0.4) (layer "F.Cu") (net 24))
@@
   (segment (start 166.385 120.005) (end 166.385 118.125) (width 0.4) (layer "F.Cu") (net 24))
   (segment (start 106.68 87.63) (end 99.314 87.63) (width 1) (layer "F.Cu") (net 24))
+  (segment (start 90.932 106.68) (end 90.932 106.538) (width 0.4) (layer "F.Cu") (net 24))
   (segment (start 94.63 133.365) (end 94.615 133.35) (width 0.4) (layer "F.Cu") (net 24))
   (segment (start 180.355 103.109) (end 180.594 102.87) (width 0.275) (layer "F.Cu") (net 24))
@@
   (via (at 193.675 118.11) (size 0.8) (drill 0.4) (layers "F.Cu" "B.Cu") (net 24))
   (via (at 99.314 87.63) (size 0.8) (drill 0.4) (layers "F.Cu" "B.Cu") (net 24))
-  (via (at 76.157265 103.601396) (size 0.8) (drill 0.4) (layers "F.Cu" "B.Cu") (net 24))
   (via (at 178.562 118.11) (size 0.8) (drill 0.4) (layers "F.Cu" "B.Cu") (net 24))
   (via (at 185.674 133.35) (size 0.8) (drill 0.4) (layers "F.Cu" "B.Cu") (net 24))
@@
   (via (at 119.126 87.63) (size 0.8) (drill 0.4) (layers "F.Cu" "B.Cu") (net 24))
   (via (at 138.43 102.87) (size 0.8) (drill 0.4) (layers "F.Cu" "B.Cu") (net 24))
+  (via (at 76.157265 103.601396) (size 0.8) (drill 0.4) (layers "F.Cu" "B.Cu") (net 24))
   (via (at 193.675 133.35) (size 0.8) (drill 0.4) (layers "F.Cu" "B.Cu") (net 24))
   (via (at 130.81 133.35) (size 0.8) (drill 0.4) (layers "F.Cu" "B.Cu") (net 24))
@@
   (segment (start 191.135 122.555) (end 185.42 122.555) (width 0.4) (layer "F.Cu") (net 65))
   (via (at 174.625 121.92) (size 0.8) (drill 0.4) (layers "F.Cu" "B.Cu") (net 65))
-  (segment (start 172.73 104.765) (end 172.735 104.765) (width 0.4) (layer "B.Cu") (net 65))
   (segment (start 172.085 105.41) (end 172.73 104.765) (width 0.4) (layer "B.Cu") (net 65))
   (segment (start 172.085 122.555) (end 172.085 105.41) (width 0.4) (layer "B.Cu") (net 65))
+  (segment (start 173.99 122.555) (end 172.085 122.555) (width 0.4) (layer "B.Cu") (net 65))
   (segment (start 174.625 121.92) (end 173.99 122.555) (width 0.4) (layer "B.Cu") (net 65))
-  (segment (start 173.99 122.555) (end 172.085 122.555) (width 0.4) (layer "B.Cu") (net 65))
+  (segment (start 172.73 104.765) (end 172.735 104.765) (width 0.4) (layer "B.Cu") (net 65))
   (segment (start 175.26 99.06) (end 195.58 99.06) (width 0.4) (layer "F.Cu") (net 66))
   (segment (start 196.1515 127.9525) (end 196.1515 124.3965) (width 0.4) (layer "F.Cu") (net 66))

Commit message: Connect RCLKs together and update doc
Connections:
- R1 pad 1: unconnected-(R1-Pad1) -> Net-(U7111-Pad11)
Routing:
- net GND: track 827.3 -> 812.0 mm
- net VCC: track 724.2 -> 726.7 mm
- net Net-(U7110-Pad12): track 206.3 -> 207.0 mm
- net /DRQ3: track 51.5 -> 50.9 mm

Commit message: Disconnect RCLKs in favor of different idea
Connections:
- U7110 pad 2: Net-(U7110-Pad2) -> Net-(U7116-Pad12)
- U7112 pad 11: Net-(U7110-Pad2) -> Net-(U7116-Pad12)
- U7116 pad 12: Net-(U7110-Pad12) -> Net-(U7116-Pad12)
- U7117 pad 12: Net-(U7110-Pad12) -> Net-(U7116-Pad12)
Routing:
- net Net-(U7116-Pad12): track 0.00 -> 111.3 mm, vias 0 -> 6
- net Net-(U7110-Pad12): track 207.0 -> 135.3 mm, vias 9 -> 5
- net Net-(U7110-Pad2): track 25.4 -> 0.00 mm, vias 2 -> 0
- net Net-(U7110-Pad1): track 33.6 -> 34.8 mm
