File: EDA/ISA-Card/ISA-Card.kicad_pcb (KiCad board)
At the start: 2 copper layers, 138.4 x 98.4 mm, 53 parts, among them U7101 74HCT245, U7102 74HCT244, U7104 74HCT138, U7105 74HCT138, U7106 74LS08, U7107 74LS32, U7108 74LS32, U7109 74HC368, U7110 74HC04, U7111 74HC125, U7112 74HC74, U7113 74HC74, U7114 74HC4024, U7115 74HC4024, U7116 74HC595, U7117 74HC595, U7118 74HC595, U7119 8251, U7120 26LS31, U7121 26LS32, X2 Conn_02x04_Counter_Clockwise, X3 DB15_Female, X5 Conn_02x08_Counter_Clockwise

Commit message: cleanup
Routing:
- net GND: vias 26 -> 25
Changed lines of the file:
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@@
   (paper "USLetter")
   (title_block
-    (title "Monster Floppy Disk Controller")
-    (date "2021-12-02")
-    (rev "1.0")
-    (company "Designed by Sergey Kiselev")
-    (comment 2 "Licensed under CERN-OHL-S: https://cern-ohl.web.cern.ch")
-    (comment 3 "Documentation and design files: https://github.com/skiselev/monster-fdc")
-    (comment 4 "Monster Floppy Disk Controller is an open source hardware project")
+    (title "Philips CM-153 LMSI Reproduction Card")
+    (date "2022-08-22")
+    (rev "alpha")
+    (company "Shelby Jueden (Tech Tangents)")
+    (comment 1 "Philips CM-153 LMSI Reproduction Card")
+    (comment 2 "Source Repository and Reference Material: https://github.com/AkBKukU/CM153-Repro")
+    (comment 3 "Licensed under CERN-OHL-S: https://cern-ohl.web.cern.ch")
   )
   (layers
@@
       (layer "B.Paste" (type "Bottom Solder Paste"))
       (layer "B.SilkS" (type "Bottom Silk Screen"))
-      (copper_finish "None")
+      (copper_finish "HAL SnPb")
       (dielectric_constraints no)
+      (edge_connector bevelled)
     )
     (pad_to_mask_clearance 0)
@@
   (segment (start 123.82 70.475) (end 123.82 68.585) (width 0.275) (layer "F.Cu") (net 24))
   (via (at 193.675 102.87) (size 0.8) (drill 0.4) (layers "F.Cu" "B.Cu") (net 24))
-  (via (at 185.674 133.35) (size 0.8) (drill 0.4) (layers "F.Cu" "B.Cu") (net 24))
   (via (at 170.434 118.11) (size 0.8) (drill 0.4) (layers "F.Cu" "B.Cu") (net 24))
   (via (at 125.73 87.63) (size 0.8) (drill 0.4) (layers "F.Cu" "B.Cu") (net 24))
@@
   (segment (start 189.23 93.345) (end 189.23 81.915) (width 0.275) (layer "B.Cu") (net 136))
   (segment (start 180.96 61.58) (end 180.975 61.595) (width 0.275) (layer "B.Cu") (net 136))
-  (segment (start 117.348 86.36) (end 117.158489 86.549511) (width 0.4) (layer "F.Cu") (net 137))
   (segment (start 152.4 77.47) (end 140.335 77.47) (width 0.4) (layer "F.Cu") (net 137))
   (segment (start 86.36 85.725) (end 102.87 85.725) (width 0.275) (layer "F.Cu") (net 137))
   (segment (start 103.694511 86.549511) (end 102.87 85.725) (width 0.4) (layer "F.Cu") (net 137))
+  (segment (start 117.158489 86.549511) (end 103.694511 86.549511) (width 0.4) (layer "F.Cu") (net 137))
   (segment (start 158.75 80.645) (end 152.4 80.645) (width 0.4) (layer "F.Cu") (net 137))
   (segment (start 140.335 77.47) (end 117.475 77.47) (width 0.4) (layer "F.Cu") (net 137))
+  (segment (start 117.348 86.36) (end 117.158489 86.549511) (width 0.4) (layer "F.Cu") (net 137))
   (segment (start 158.765 81.915) (end 158.765 80.66) (width 0.4) (layer "F.Cu") (net 137))
-  (segment (start 117.158489 86.549511) (end 103.694511 86.549511) (width 0.4) (layer "F.Cu") (net 137))
   (segment (start 158.765 80.66) (end 158.75 80.645) (width 0.4) (layer "F.Cu") (net 137))
   (via (at 152.4 80.645) (size 0.8) (drill 0.4) (layers "F.Cu" "B.Cu") (net 137))

Commit message: Added Philips Custom Mounting Holes
Parts:
- removed HOLE2 (x3): HOLE, MountingHole:MountingHole_3.2mm_M3_Pad_Via
- added REF**: Bracket Mount, Philips-Shapes:Bracket Mount, F.Cu at (206.4, 66.7)
- added REF**: Wide Mounting Hole, Philips-Shapes:Wide Mounting Hole, F.Cu at (79.5, 57.6)
- added REF**: Mounting Hole, Philips-Shapes:Mounting Hole, F.Cu at (199.8, 85.7)
